Commit message: feat: hand-eye calibration complete (project 1 stage B)
- 16_capture_calibration.py: headless capture with HTTP preview server
  (http://192.168.0.2:8090), camera bandwidth fix (front MJPG, handeye
  lower res), sys import fix, terminal ENTER/r/q + web buttons
- 17_handeye_calibrate.py: board-side calibration (OpenCV 4.13 has
  calibrateHandEye; PC OpenCV 5.0 removed it) with URDF FK parser
- calib_data: 15 samples, all 88 corners detected on both cameras
- calib_out: intrinsics + extrinsics JSON
  handeye: reproj 0.46px, camera->gripper_frame_link
  front:   reproj 6.42px, camera->base_link (wide angle, optimize later)
- so101.urdf: added handeye_camera_link + front_camera_link with real
  calibrated extrinsics (fixed joints)

File: ros2_ws/src/so101_description/urdf/so101.urdf (robot description, URDF)
Before this commit: robot so101_new_calib, 8 links, 7 joints
Links:
- added link front_camera_link
- added link handeye_camera_link
Joints:
- added joint front_camera_joint: type fixed, parent base_link, child front_camera_link, origin xyz=-0.036676 -0.101546 0.011455 rpy=0.121616 -0.299542 -1.591590
- added joint handeye_camera_joint: type fixed, parent gripper_frame_link, child handeye_camera_link, origin xyz=-0.003490 0.063697 -0.091141 rpy=-0.427446 -0.058455 2.988576

Commit message: fix: front camera recalibration v2 (correct eye-to-hand data)
- front intrinsics v2: 6.42px -> 0.74px (handheld board, fills frame)
- front extrinsic v2: correct data condition (checkerboard on wrist moves
  with arm, camera fixed), 15/15 poses usable, t=(-36,-66,109)mm
- 18_capture_front_intrinsics.py: front-only capture with HTTP preview
- front_extrinsic_v2.py: recompute extrinsic with new intrinsics
- so101.urdf: front_camera_joint updated with v2 extrinsic

File: ros2_ws/src/so101_description/urdf/so101.urdf (robot description, URDF)
Before this commit: robot so101_new_calib, 10 links, 9 joints
Joints:
- joint front_camera_joint: origin xyz=-0.036676 -0.101546 0.011455 rpy=0.121616 -0.299542 -1.591590 -> xyz=-0.036287 -0.066093 0.108881 rpy=-0.703520 -0.876047 -0.842733

Commit message: fix: front camera extrinsic via geometric single-shot method
- Correct convention: solvePnP returns cam-in-board, use T_cam2base =
  T_board2cam @ T_board2base (no inverse); camera Z axis flipped via Ry(pi)
- Measured board center (0.293, 0, 0); camera at (-4, -52, +383)mm
- Live verify: yellow object localized to (13.8, 13.1)cm in workspace
- 19_locate_object.py now uses geometric extrinsic
- so101.urdf front_camera_joint updated to v3

File: ros2_ws/src/so101_description/urdf/so101.urdf (robot description, URDF)
Before this commit: robot so101_new_calib, 10 links, 9 joints
Joints:
- joint front_camera_joint: origin xyz=-0.036287 -0.066093 0.108881 rpy=-0.703520 -0.876047 -0.842733 -> xyz=-0.004000 -0.052000 0.383000 rpy=2.835714 -0.081059 -3.128554

Commit message: fix: front camera extrinsic FINAL - correct R.T convention
- Root cause: T_b2base extra translation bug; correct combo is
  T_cam2base = [R.T | -R.T t] (objp built directly in base frame)
- Self-check PASSES: board center (0.293,0,0.003) back-projects to
  (29.3, 0.0, 0.3)cm exactly
- Camera at (16, 0, 37)cm, optical axis down
- Live: yellow object at (35.1, -22.2)cm stable
- so101.urdf front_camera_joint updated
- front_geometric_calib_v2.py: fixed-orientation geometric calibration

File: ros2_ws/src/so101_description/urdf/so101.urdf (robot description, URDF)
Before this commit: robot so101_new_calib, 10 links, 9 joints
Joints:
- joint front_camera_joint: origin xyz=-0.004000 -0.052000 0.383000 rpy=2.835714 -0.081059 -3.128554 -> xyz=0.160433 -0.000879 0.367050 rpy=2.740071 0.112603 1.567879
